File: Power-Conversion.brd (EAGLE design)
At the start: 252.4 x 86.3 mm, 43 parts, among them Q1 SUM90P10-19L, U7 LM2678

Commit message: Added new connectors for 8th bricks
Parts:
- removed U$11, U$12, U$17: POWER_BRICK_CONNECTORS(2X15), MotherBoardParts2:POWER_BRICK_CONNECTORS(2X15)
- removed U$13, U$14, U$15: POWER_BRICK_CONNECTORS(2X6), MotherBoardParts2:POWER_BRICK_CONNECTORS(2X6)
- added U$20, U$21, U$22, U$23: BRICK_TO_POWER_DIST_WHOLE, MotherBoardParts2:BRICK_TO_POWER_DIST_WHOLE
- added U$24: DIODE, diode:DIODE
Connections:
- new net +12V_4: U$23.+12V1, U$23.+12V10, U$23.+12V2, U$23.+12V3, U$23.+12V4, U$23.+12V5, U$23.+12V6, U$23.+12V7, U$23.+12V8, U$23.+12V9, U$24.IN1, U$24.IN2
- new net V-: U$20.48V_GND1, U$20.48V_GND2, U$20.48V_GND3, U$20.48V_GND4, U$21.48V_GND1, U$21.48V_GND2, U$21.48V_GND3, U$21.48V_GND4, U$22.48V_GND1, U$22.48V_GND2, U$22.48V_GND3, U$22.48V_GND4, U$23.48V_GND1, U$23.48V_GND2, U$23.48V_GND3, U$23.48V_GND4
- new net VCC: U$20.+48V1, U$20.+48V2, U$20.+48V3, U$20.+48V4, U$21.+48V1, U$21.+48V2, U$21.+48V3, U$21.+48V4, U$22.+48V1, U$22.+48V2, U$22.+48V3, U$22.+48V4, U$23.+48V1, U$23.+48V2, U$23.+48V3, U$23.+48V4
- net +12V: now also U$24.OUT
- net +12V_1: now also U$20.+12V1, U$20.+12V10, U$20.+12V2, U$20.+12V3, U$20.+12V4, U$20.+12V5, U$20.+12V6, U$20.+12V7, U$20.+12V8, U$20.+12V9; no longer U$17.P$1, U$17.P$16, U$17.P$17, U$17.P$18, U$17.P$19, U$17.P$2, U$17.P$20, U$17.P$21, U$17.P$22, U$17.P$3, U$17.P$4, U$17.P$5, U$17.P$6, U$17.P$7
- net +12V_2: now also U$21.+12V1, U$21.+12V10, U$21.+12V2, U$21.+12V3, U$21.+12V4, U$21.+12V5, U$21.+12V6, U$21.+12V7, U$21.+12V8, U$21.+12V9; no longer U$11.P$1, U$11.P$16, U$11.P$17, U$11.P$18, U$11.P$19, U$11.P$2, U$11.P$20, U$11.P$21, U$11.P$22, U$11.P$3, U$11.P$4, U$11.P$5, U$11.P$6, U$11.P$7
- net +12V_3: now also U$22.+12V1, U$22.+12V10, U$22.+12V2, U$22.+12V3, U$22.+12V4, U$22.+12V5, U$22.+12V6, U$22.+12V7, U$22.+12V8, U$22.+12V9; no longer U$12.P$1, U$12.P$16, U$12.P$17, U$12.P$18, U$12.P$19, U$12.P$2, U$12.P$20, U$12.P$21, U$12.P$22, U$12.P$3, U$12.P$4, U$12.P$5, U$12.P$6, U$12.P$7
- net +48V_SNS: no longer U$13.P$1, U$13.P$2, U$13.P$7, U$13.P$8, U$14.P$1, U$14.P$2, U$14.P$7, U$14.P$8, U$15.P$1, U$15.P$2, U$15.P$7, U$15.P$8
- net 48V_GND: no longer U$13.P$10, U$13.P$3, U$13.P$4, U$13.P$9, U$14.P$10, U$14.P$3, U$14.P$4, U$14.P$9, U$15.P$10, U$15.P$3, U$15.P$4, U$15.P$9
- net GND: now also U$20.D_GND, U$20.GND1, U$20.GND10, U$20.GND2, U$20.GND3, U$20.GND4, U$20.GND5, U$20.GND6, U$20.GND7, U$20.GND8, U$20.GND9, U$21.D_GND, U$21.GND1, U$21.GND10, U$21.GND2, U$21.GND3, U$21.GND4, U$21.GND5, U$21.GND6, U$21.GND7, U$21.GND8, U$21.GND9, U$22.D_GND, U$22.GND1, U$22.GND10, U$22.GND2, U$22.GND3, U$22.GND4, U$22.GND5, U$22.GND6, U$22.GND7, U$22.GND8, U$22.GND9, U$23.D_GND, U$23.GND1, U$23.GND10, U$23.GND2, U$23.GND3, U$23.GND4, U$23.GND5, U$23.GND6, U$23.GND7, U$23.GND8, U$23.GND9; no longer U$11.P$10, U$11.P$11, U$11.P$12, U$11.P$13, U$11.P$14, U$11.P$15, U$11.P$24, U$11.P$25, U$11.P$26, U$11.P$27, U$11.P$28, U$11.P$29, U$11.P$30, U$11.P$9, U$12.P$10, U$12.P$11, U$12.P$12, U$12.P$13, U$12.P$14, U$12.P$15, U$12.P$24, U$12.P$25, U$12.P$26, U$12.P$27, U$12.P$28, U$12.P$29, U$12.P$30, U$12.P$9, U$13.P$5, U$14.P$5, U$15.P$5, U$17.P$10, U$17.P$11, U$17.P$12, U$17.P$13, U$17.P$14, U$17.P$15, U$17.P$24, U$17.P$25, U$17.P$26, U$17.P$27, U$17.P$28, U$17.P$29, U$17.P$30, U$17.P$9
- net ON/OFF: now also U$20.ON/OFF, U$21.ON/OFF, U$22.ON/OFF, U$23.ON/OFF; no longer U$13.P$11, U$14.P$11, U$15.P$11
- net SCL: now also U$20.SCL, U$21.SCL, U$22.SCL, U$23.SCL; no longer U$13.P$12, U$14.P$12, U$15.P$12
- net SDA: now also U$20.SDA, U$21.SDA, U$22.SDA, U$23.SDA; no longer U$13.P$6, U$14.P$6, U$15.P$6

Commit message: Initial layout of parts has begun.  Still need to reduce down the size a lot...
Parts:
- added J3, J4: (no value), SparkFun-Connectors:BANANA_CONN
- added R15, R5: 0R, resistor:R0603
- added U$11: T2I5P, BackplaneParts:T2I5P
- added U$12: T2I, BackplaneParts:T2I
- moved U$24 280.1 mm to (88.9, 78.7), turned to 180 degrees
- moved U$23 226.4 mm to (55.9, 67.3)
- moved U$22 225.2 mm to (94.0, 67.3)
- moved U$21 223.9 mm to (132.1, 67.3)
- moved U$20 222.6 mm to (170.2, 67.3)
- moved R1 122.6 mm to (88.6, 115.6), turned to 0 degrees
- moved U$4 119.3 mm to (88.9, 119.4), turned to 270 degrees
- moved U$6 117.6 mm to (92.7, 119.4), turned to 270 degrees
- moved R2 112.5 mm to (92.7, 115.6), turned to 0 degrees
- moved C3 70.0 mm to (13.5, 128.3)
- moved R11 70.0 mm to (51.8, 129.8)
- moved C10 70.0 mm to (40.6, 127.3)
- moved C11 70.0 mm to (39.1, 115.6)
- moved C12 70.0 mm to (32.3, 115.6)
- moved C13 70.0 mm to (46.2, 115.6)
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Connections:
- removed net 12V: U$16.P$1, U$16.P$2, U$16.P$3, U$8.P$1, U$8.P$10, U$8.P$11, U$8.P$12, U$8.P$13, U$8.P$14, U$8.P$15, U$8.P$16, U$8.P$17, U$8.P$18, U$8.P$19, U$8.P$2, U$8.P$20, U$8.P$21, U$8.P$22, U$8.P$23, U$8.P$24, U$8.P$25, U$8.P$26, U$8.P$27, U$8.P$28, U$8.P$29, U$8.P$3, U$8.P$30, U$8.P$31, U$8.P$32, U$8.P$33, U$8.P$34, U$8.P$35, U$8.P$36, U$8.P$37, U$8.P$38, U$8.P$39, U$8.P$4, U$8.P$40, U$8.P$41, U$8.P$42, U$8.P$43, U$8.P$44, U$8.P$45, U$8.P$46, U$8.P$47, U$8.P$48, U$8.P$49, U$8.P$5, U$8.P$50, U$8.P$6, U$8.P$7, U$8.P$8, U$8.P$9
- new net N$2: U$12.1
- new net N$3: U$12.2
- new net SCL1: R5.1, U$20.SCL, U$21.SCL, U$22.SCL
- new net SCL4: U$23.SCL
- new net SDA1: R15.1, U$20.SDA, U$21.SDA, U$22.SDA
- new net SDA4: U$23.SDA
- net +12V: now also U$16.P$1, U$16.P$2, U$16.P$3, U$8.P$1, U$8.P$10, U$8.P$11, U$8.P$12, U$8.P$13, U$8.P$14, U$8.P$15, U$8.P$16, U$8.P$17, U$8.P$18, U$8.P$19, U$8.P$2, U$8.P$20, U$8.P$21, U$8.P$22, U$8.P$23, U$8.P$24, U$8.P$25, U$8.P$26, U$8.P$27, U$8.P$28, U$8.P$29, U$8.P$3, U$8.P$30, U$8.P$31, U$8.P$32, U$8.P$33, U$8.P$34, U$8.P$35, U$8.P$36, U$8.P$37, U$8.P$38, U$8.P$39, U$8.P$4, U$8.P$40, U$8.P$41, U$8.P$42, U$8.P$43, U$8.P$44, U$8.P$45, U$8.P$46, U$8.P$47, U$8.P$48, U$8.P$49, U$8.P$5, U$8.P$50, U$8.P$6, U$8.P$7, U$8.P$8, U$8.P$9
- net +48V: now also J4.P$1
- net +48V_RAW: now also J3.P$1
- net +5V: now also U$11.P$5, U$11.P$6
- net GND: now also U$11.P$2, U$11.P$3
- net SCL: now also R5.2, U$12.4; no longer U$20.SCL, U$21.SCL, U$22.SCL, U$23.SCL
- net SDA: now also R15.2, U$12.3; no longer U$20.SDA, U$21.SDA, U$22.SDA, U$23.SDA
Routing:
- net GND: track 53.8 -> 0.87 mm
- net +5V: track 50.8 -> 0.83 mm, vias 2 -> 0
- net +12V: track 47.3 -> 0.00 mm, vias 2 -> 0
- net N$36: track 26.2 -> 0.00 mm
- net N$10: track 23.5 -> 0.00 mm
- net ONOFF: track 10.6 -> 0.00 mm
- net N$5: track 9.96 -> 0.00 mm
- net 48V_GND: track 9.66 -> 0.00 mm, vias 2 -> 0
- net N$25: track 6.93 -> 0.00 mm
- net 48_I_ANALOG: track 6.62 -> 0.00 mm
- net N$40: track 4.75 -> 0.00 mm
- net N$39: track 4.50 -> 0.00 mm
- net N$9: track 2.20 -> 0.00 mm
- added copper zone on layer 1, net +12V_1
- added copper zone on layer 1, net +12V_2
- added copper zone on layer 1, net +12V_3
- added copper zone on layer 1, net +12V_4
- added copper zone on layer 16, net GND
- removed copper zone on layer 1, net +5V
- removed copper zone on layer 16, net 48V_GND
- removed copper zone on layer 1, net GND
Other:
- board size 252.4 x 86.3 mm -> 218.4 x 101.6 mm
