File: Power-Conversion.brd (EAGLE design)
At the start: 182.9 x 114.3 mm, 49 parts, among them Q1 SUM90P10-19L, U7 LM2678

Commit message: Some changes for second round of manufacturing
Parts:
- added J4, J7: (no value), SparkFun-Connectors:BANANA_CONN
Connections:
- net +12V: now also J4.P$1; no longer U$8.P$4, U$8.P$5, U$8.P$6
- net GND: now also J7.P$1; no longer U$8.P$10, U$8.P$11, U$8.P$12
Routing:
- net 48_I_ANALOG: track 268.0 -> 275.0 mm
- added copper zone on layer 16, net N$4
Changed lines of the file:
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@@
 <setting verticaltext="up"/>
 </settings>
-<grid distance="7" unitdist="mil" unit="mil" style="lines" multiple="1" display="yes" altdistance="5" altunitdist="mil" altunit="mil"/>
+<grid distance="25" unitdist="mil" unit="mil" style="lines" multiple="1" display="yes" altdistance="5" altunitdist="mil" altunit="mil"/>
 <layers>
 <layer number="1" name="Top" color="4" fill="1" visible="yes" active="yes"/>
@@
 <layer number="27" name="tValues" color="7" fill="1" visible="yes" active="yes"/>
 <layer number="28" name="bValues" color="7" fill="1" visible="yes" active="yes"/>
-<layer number="29" name="tStop" color="7" fill="3" visible="yes" active="yes"/>
-<layer number="30" name="bStop" color="7" fill="6" visible="yes" active="yes"/>
-<layer number="31" name="tCream" color="7" fill="4" visible="yes" active="yes"/>
-<layer number="32" name="bCream" color="7" fill="5" visible="yes" active="yes"/>
-<layer number="33" name="tFinish" color="6" fill="3" visible="yes" active="yes"/>
-<layer number="34" name="bFinish" color="6" fill="6" visible="yes" active="yes"/>
-<layer number="35" name="tGlue" color="7" fill="4" visible="yes" active="yes"/>
-<layer number="36" name="bGlue" color="7" fill="5" visible="yes" active="yes"/>
+<layer number="29" name="tStop" color="7" fill="3" visible="no" active="yes"/>
+<layer number="30" name="bStop" color="7" fill="6" visible="no" active="yes"/>
+<layer number="31" name="tCream" color="7" fill="4" visible="no" active="yes"/>
+<layer number="32" name="bCream" color="7" fill="5" visible="no" active="yes"/>
+<layer number="33" name="tFinish" color="6" fill="3" visible="no" active="yes"/>
+<layer number="34" name="bFinish" color="6" fill="6" visible="no" active="yes"/>
+<layer number="35" name="tGlue" color="7" fill="4" visible="no" active="yes"/>
+<layer number="36" name="bGlue" color="7" fill="5" visible="no" active="yes"/>
 <layer number="37" name="tTest" color="7" fill="1" visible="yes" active="yes"/>
 <layer number="38" name="bTest" color="7" fill="1" visible="yes" active="yes"/>
@@
 <layer number="42" name="bRestrict" color="1" fill="10" visible="yes" active="yes"/>
 <layer number="43" name="vRestrict" color="2" fill="10" visible="yes" active="yes"/>
-<layer number="44" name="Drills" color="7" fill="1" visible="yes" active="yes"/>
-<layer number="45" name="Holes" color="7" fill="1" visible="yes" active="yes"/>
+<layer number="44" name="Drills" color="7" fill="1" visible="no" active="yes"/>
+<layer number="45" name="Holes" color="7" fill="1" visible="no" active="yes"/>
 <layer number="46" name="Milling" color="3" fill="1" visible="yes" active="yes"/>
 <layer number="47" name="Measures" color="7" fill="1" visible="yes" active="yes"/>
@@
 <element name="JP2" library="pinhead" library_urn="urn:adsk.eagle:library:325" package="1X01" package3d_urn="urn:adsk.eagle:package:22485/2" value="" x="20.955" y="9.779"/>
 <element name="J3" library="SparkFun-Connectors" package="BANANA_CONN" value="" x="131.953" y="5.334"/>
+<element name="J4" library="SparkFun-Connectors" package="BANANA_CONN" value="" x="165.735" y="104.775"/>
+<element name="J7" library="SparkFun-Connectors" package="BANANA_CONN" value="" x="165.735" y="92.71"/>
 </elements>
 <signals>
@@
 <contactref element="U$11" pad="P$3"/>
 <contactref element="U$11" pad="P$2"/>
-<polygon width="0.1524" layer="16" rank="6">
+<polygon width="0.1524" layer="16" isolate="0.508" rank="6">
 <vertex x="0" y="92.71"/>
 <vertex x="39.37" y="92.71"/>
@@
 <via x="181.356" y="24.384" extent="1-16" drill="0.35"/>
 <via x="180.086" y="31.242" extent="1-16" drill="0.35"/>
-<polygon width="0.4064" layer="16">
-<vertex x="28.448" y="96.52"/>
-<vertex x="44.323" y="96.52"/>
-<vertex x="44.323" y="100.076"/>
-<vertex x="19.558" y="100.33"/>
-<vertex x="19.558" y="92.456"/>
-<vertex x="19.304" y="92.202"/>
-<vertex x="28.448" y="92.202"/>
-</polygon>
 <wire x1="19.05" y1="50.247" x2="19.05" y2="46.736" width="1.27" layer="1"/>
 <via x="19.05" y="46.736" extent="1-16" drill="0.65" diameter="1.3"/>
@@
 <contactref element="U$8" pad="P$21"/>
 <contactref element="U$8" pad="P$55"/>
-<contactref element="U$8" pad="P$12"/>
-<contactref element="U$8" pad="P$11"/>
-<contactref element="U$8" pad="P$10"/>
 <wire x1="181.356" y1="27.94" x2="180.086" y2="29.21" width="0.6096" layer="1"/>
 <wire x1="180.086" y1="29.21" x2="180.086" y2="31.242" width="0.6096" layer="1"/>
@@
 <wire x1="160.147" y1="15.836" x2="159.551" y2="15.24" width="0.6096" layer="16"/>
 <wire x1="159.551" y1="15.24" x2="158.076" y2="15.24" width="0.6096" layer="16"/>
+<contactref element="J7" pad="P$1"/>
 </signal>
 <signal name="N$9">
@@
 <contactref element="U$8" pad="P$109"/>
 <contactref element="U$8" pad="P$124"/>
-<contactref element="U$8" pad="P$4"/>
-<contactref element="U$8" pad="P$6"/>
-<contactref element="U$8" pad="P$5"/>
-<polygon width="0.4064" layer="1">
-<vertex x="36.322" y="96.774"/>
-<vertex x="59.055" y="96.774"/>
-<vertex x="59.055" y="84.582"/>
-<vertex x="55.245" y="84.582"/>
-<vertex x="55.245" y="94.234"/>
-<vertex x="36.322" y="94.234"/>
+<contactref element="J4" pad="P$1"/>
+<polygon width="0.1524" layer="1">
+<vertex x="120.65" y="86.36"/>
+<vertex x="120.65" y="108.585"/>
+<vertex x="169.545" y="108.585"/>
+<vertex x="169.545" y="100.965"/>
+<vertex x="128.905" y="100.965"/>
+<vertex x="125.095" y="100.965"/>
+<vertex x="125.095" y="86.36"/>
+<vertex x="125.095" y="84.455"/>
+<vertex x="120.65" y="84.455"/>
 </polygon>
 </signal>
@@
 <via x="181.4858" y="29.337" extent="1-16" drill="0.35"/>
 <wire x1="181.4858" y1="29.337" x2="181.4858" y2="98.9302" width="0.6096" layer="1"/>
-<wire x1="181.4858" y1="98.9302" x2="177.165" y2="103.251" width="0.6096" layer="1"/>
-<wire x1="177.165" y1="103.251" x2="37.973" y2="103.251" width="0.6096" layer="1"/>
-<wire x1="37.973" y1="103.251" x2="32.639" y2="97.917" width="0.6096" layer="1"/>
+<wire x1="37.973" y1="103.251" x2="37.846" y2="103.124" width="0.6096" layer="1"/>
+<wire x1="37.846" y1="103.124" x2="32.639" y2="97.917" width="0.6096" layer="1"/>
 <wire x1="153.2382" y1="15.113" x2="152.019" y2="15.113" width="0.6096" layer="16"/>
 <wire x1="152.019" y1="15.113" x2="151.638" y2="15.494" width="0.6096" layer="16"/>
@@
 <wire x1="152.781" y1="19.25208125" x2="157.988" y2="24.45908125" width="0.6096" layer="16"/>
 <wire x1="157.988" y1="24.45908125" x2="157.988" y2="24.511" width="0.6096" layer="16"/>
+<wire x1="168.656" y1="111.76" x2="181.4858" y2="98.9302" width="0.6096" layer="1"/>
+<wire x1="37.973" y1="103.251" x2="46.482" y2="111.76" width="0.6096" layer="1"/>
+<wire x1="46.482" y1="111.76" x2="168.656" y2="111.76" width="0.6096" layer="1"/>
 </signal>
 <signal name="ON/OFF">
@@
 <wire x1="18.454" y1="63.119" x2="18.415" y2="63.119" width="0.8128" layer="16"/>
 </signal>
+<signal name="N$4">
+<polygon width="0.1524" layer="16" pour="cutout">
+<vertex x="31.75" y="24.765"/>
+<vertex x="31.75" y="64.135"/>
+<vertex x="44.45" y="64.135"/>
+<vertex x="44.45" y="24.765"/>
+</polygon>
+</signal>
 </signals>
